File: schematic/nixie clock.brd (EAGLE design)
At the start: 100 x 80 mm, 57 parts, among them IC1 74141N, Q1 32,768kHz, Q2 16Mhz, T1 MPSA92, T10 MPSA92, T11 MPSA42, T12 MPSA92, T13 MPSA42, T14 MPSA92, T15 MPSA42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

Commit message: Schaltplan aktualisiert
Parts:
- removed DCF77: (no value), SparkFun-Connectors:1X03
- moved R4 6.48 mm to (26.7, 19.1)
Connections:
- net GND: no longer DCF77.3
- net N$65: no longer DCF77.2
- net VCC: no longer DCF77.1
Changed lines of the file:
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@@
 <?xml version="1.0" encoding="utf-8"?>
 <!DOCTYPE eagle SYSTEM "eagle.dtd">
-<eagle version="6.5.0">
+<eagle version="8.0.0">
 <drawing>
 <settings>
@@
 <layer number="56" name="wert" color="7" fill="1" visible="yes" active="yes"/>
 <layer number="57" name="tCAD" color="7" fill="1" visible="no" active="no"/>
-<layer number="90" name="Modules" color="5" fill="1" visible="yes" active="yes"/>
+<layer number="90" name="Modules" color="5" fill="1" visible="no" active="no"/>
 <layer number="91" name="Nets" color="2" fill="1" visible="no" active="no"/>
 <layer number="92" name="Busses" color="1" fill="1" visible="no" active="no"/>
@@
 <wire x1="100" y1="80" x2="0" y2="80" width="0" layer="20"/>
 <wire x1="0" y1="80" x2="0" y2="0" width="0" layer="20"/>
-<dimension x1="0" y1="0" x2="0" y2="72.39" x3="-6.35" y3="36.195" textsize="1.778" layer="1"/>
-<dimension x1="0" y1="0" x2="120.65" y2="0" x3="60.325" y3="-6.35" textsize="1.778" layer="1"/>
+<dimension x1="0" y1="80" x2="0" y2="29.21" x3="-6.35" y3="54.605" textsize="1.778" layer="16"/>
 </plain>
 <attributes>
@@
 <pass name="Default">
 <param name="RoutingGrid" value="50mil"/>
+<param name="AutoGrid" value="1"/>
+<param name="Efforts" value="0"/>
+<param name="TopRouterVariant" value="1"/>
 <param name="tpViaShape" value="round"/>
 <param name="PrefDir.1" value="|"/>
@@
 <element name="C1" library="SparkFun-Capacitors" package="CAP-PTH-SMALLEZ" value="22pf" x="77.47" y="44.45" rot="R270"/>
 <element name="C2" library="SparkFun-Capacitors" package="CAP-PTH-SMALLEZ" value="22pf" x="72.39" y="44.45" rot="R270"/>
-<element name="DCF77" library="SparkFun-Connectors" package="1X03" value="" x="26.67" y="29.21" rot="R180"/>
-<element name="R4" library="resistor" package="0204/7" value="1k" x="27.94" y="25.4"/>
+<element name="R4" library="resistor" package="0204/7" value="1k" x="26.67" y="19.05"/>
 <element name="BAT1" library="SparkFun-Electromechanical" package="BATTCOM_20MM_PTH" value="3V" x="44.45" y="13.97"/>
 <element name="SERIAL" library="con-lstb" package="MA04-1" value="" x="96.52" y="40.64" rot="R90">
@@
 <contactref element="C2" pad="1"/>
 <contactref element="C1" pad="1"/>
-<contactref element="DCF77" pad="3"/>
 <contactref element="BAT1" pad="2"/>
 <contactref element="SERIAL" pad="4"/>
@@
 <wire x1="81.28" y1="22.86" x2="78.74" y2="30.48" width="0" layer="19" extent="1-1"/>
 <wire x1="74.93" y1="11.43" x2="81.28" y2="22.86" width="0" layer="19" extent="1-1"/>
-<wire x1="21.59" y1="29.21" x2="21.59" y2="48.26" width="0" layer="19" extent="1-1"/>
-<wire x1="36.3" y1="13.97" x2="21.59" y2="29.21" width="0" layer="19" extent="1-1"/>
 <wire x1="96.52" y1="5.08" x2="74.93" y2="11.43" width="0" layer="19" extent="1-1"/>
-<wire x1="3.81" y1="3.81" x2="21.59" y2="29.21" width="0" layer="19" extent="1-1"/>
+<wire x1="36.3" y1="13.97" x2="36.83" y2="48.26" width="0" layer="19" extent="1-1"/>
+<wire x1="3.81" y1="3.81" x2="36.3" y2="13.97" width="0" layer="19" extent="1-1"/>
 <wire x1="-18.4912" y1="-4.8006" x2="3.81" y2="3.81" width="0" layer="19" extent="1-1"/>
 <wire x1="-29.9212" y1="-4.8006" x2="-18.4912" y2="-4.8006" width="0" layer="19" extent="1-1"/>
@@
 <contactref element="U1" pad="20"/>
 <contactref element="U1" pad="21"/>
-<contactref element="DCF77" pad="1"/>
 <contactref element="R4" pad="2"/>
 <contactref element="R11" pad="1"/>
@@
 <wire x1="88.9" y1="12.7" x2="88.9" y2="15.24" width="0" layer="19" extent="1-1"/>
 <wire x1="69.85" y1="11.43" x2="76.2" y2="22.86" width="0" layer="19" extent="1-1"/>
-<wire x1="31.75" y1="25.4" x2="69.85" y2="11.43" width="0" layer="19" extent="1-1"/>
-<wire x1="26.67" y1="29.21" x2="31.75" y2="25.4" width="0" layer="19" extent="1-1"/>
-<wire x1="3.81" y1="8.89" x2="26.67" y2="29.21" width="0" layer="19" extent="1-1"/>
+<wire x1="30.48" y1="19.05" x2="69.85" y2="11.43" width="0" layer="19" extent="1-1"/>
+<wire x1="3.81" y1="8.89" x2="30.48" y2="19.05" width="0" layer="19" extent="1-1"/>
 </signal>
 <signal name="N$2">
@@
 <signal name="N$65">
 <contactref element="U1" pad="23"/>
-<contactref element="DCF77" pad="2"/>
 <contactref element="R4" pad="1"/>
 <contactref element="R22" pad="2"/>
-<wire x1="24.13" y1="25.4" x2="83.82" y2="22.86" width="0" layer="19" extent="1-1"/>
-<wire x1="24.13" y1="29.21" x2="24.13" y2="25.4" width="0" layer="19" extent="1-1"/>
-<wire x1="-34.29" y1="-19.05" x2="24.13" y2="25.4" width="0" layer="19" extent="1-1"/>
+<wire x1="22.86" y1="19.05" x2="83.82" y2="22.86" width="0" layer="19" extent="1-1"/>
+<wire x1="-34.29" y1="-19.05" x2="22.86" y2="19.05" width="0" layer="19" extent="1-1"/>
 </signal>
 <signal name="N$48">
