File: schematic/nixie clock.sch (EAGLE design)
At the start: 57 parts, among them IC1 74141N, Q1 32,768kHz, Q2 16Mhz, T1 MPSA92, T10 MPSA92, T11 MPSA42, T12 MPSA92, T13 MPSA42, T14 MPSA92, T15 MPSA42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

Commit message: Schaltplan aktualisiert
Parts:
- removed DCF77: (no value), SparkFun-Connectors:M03PTH
Connections:
- net GND: no longer DCF77.3
- net N$65: no longer DCF77.2
- net VCC: no longer DCF77.1
Other:
- moved on the sheet: R4
Changed lines of the file:
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@@
 <?xml version="1.0" encoding="utf-8"?>
 <!DOCTYPE eagle SYSTEM "eagle.dtd">
-<eagle version="6.5.0">
+<eagle version="6.6.0">
 <drawing>
 <settings>
@@
 <part name="C2" library="SparkFun-Capacitors" deviceset="CAP" device="EZ" value="22pf"/>
 <part name="GND14" library="supply1" deviceset="GND" device=""/>
-<part name="DCF77" library="SparkFun-Connectors" deviceset="M03" device="PTH"/>
 <part name="R4" library="resistor" deviceset="R-EU_" device="0204/7" value="1k"/>
 <part name="SUPPLY5" library="supply2" deviceset="VCC" device=""/>
-<part name="GND15" library="supply1" deviceset="GND" device=""/>
 <part name="SUPPLY6" library="supply2" deviceset="VCC" device=""/>
 <part name="BAT1" library="SparkFun-Electromechanical" deviceset="BATTERY" device="20PTH" value="3V"/>
@@
 </instance>
 <instance part="GND14" gate="1" x="-116.84" y="86.36" rot="R270"/>
-<instance part="DCF77" gate="G$1" x="-40.64" y="132.08" rot="R270"/>
-<instance part="R4" gate="G$1" x="-50.8" y="119.38" rot="R90"/>
-<instance part="SUPPLY5" gate="G$1" x="-43.18" y="119.38" rot="R180"/>
-<instance part="GND15" gate="1" x="-38.1" y="119.38"/>
+<instance part="R4" gate="G$1" x="-50.8" y="114.3"/>
+<instance part="SUPPLY5" gate="G$1" x="-43.18" y="114.3" rot="R270"/>
 <instance part="SUPPLY6" gate="G$1" x="-35.56" y="99.06" rot="R270"/>
 <instance part="BAT1" gate="G$1" x="-25.4" y="137.16" smashed="yes" rot="R90">
@@
 </segment>
 <segment>
-<pinref part="GND15" gate="1" pin="GND"/>
-<pinref part="DCF77" gate="G$1" pin="3"/>
-<wire x1="-38.1" y1="124.46" x2="-38.1" y2="121.92" width="0.1524" layer="91"/>
-</segment>
-<segment>
 <pinref part="SERIAL" gate="1" pin="4"/>
 <pinref part="GND16" gate="1" pin="GND"/>
@@
 <segment>
 <pinref part="SUPPLY5" gate="G$1" pin="VCC"/>
-<pinref part="DCF77" gate="G$1" pin="1"/>
-<wire x1="-43.18" y1="124.46" x2="-43.18" y2="121.92" width="0.1524" layer="91"/>
 <pinref part="R4" gate="G$1" pin="2"/>
-<wire x1="-50.8" y1="124.46" x2="-43.18" y2="124.46" width="0.1524" layer="91"/>
-<junction x="-43.18" y="124.46"/>
 </segment>
 <segment>
@@
 <segment>
 <pinref part="U1" gate="G$1" pin="PC0(ADC0)"/>
-<wire x1="-55.88" y1="114.3" x2="-50.8" y2="114.3" width="0.1524" layer="91"/>
-<pinref part="DCF77" gate="G$1" pin="2"/>
-<wire x1="-50.8" y1="114.3" x2="-40.64" y2="114.3" width="0.1524" layer="91"/>
-<wire x1="-40.64" y1="114.3" x2="-40.64" y2="124.46" width="0.1524" layer="91"/>
 <pinref part="R4" gate="G$1" pin="1"/>
-<junction x="-50.8" y="114.3"/>
 <pinref part="R22" gate="G$1" pin="2"/>
 <wire x1="-60.96" y1="121.92" x2="-55.88" y2="121.92" width="0.1524" layer="91"/>
