File: schematic/nixie board.brd (EAGLE design)
At the start: 100 x 72 mm, 46 parts, among them IC1 74141N, T1 MPSA42, T10 MPSA92, T11 MPSA92, T12 MPSA92, T2 MPSA42, T3 MPSA42, T4 MPSA42, T5 MPSA42, T6 MPSA42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

Commit message: added reset and elko
Parts:
- added C5: 100 µF, rcl:E2,5-6
- added R20: 10k, resistor:0204/7
- added RESET: (no value), switch-omron:B3F-10XX
- R19: device resistor:0207/2V -> resistor:0204/7
- SR33: value MCP1703-33 -> MCP1702-33
- SR50: value MCP1703-50 -> MCP1702-50
- moved SERIAL 46.8 mm to (90.6, 35.9), turned to 180 degrees
- moved R19 28.2 mm to (54.5, 23.0), turned to 0 degrees
- moved PROG 13.6 mm to (76.5, 7.01)
- moved EXT1 8.56 mm to (58.8, 32.4)
- moved EXT2 8.56 mm to (58.8, 12.1)
- moved DIGITS 8.50 mm to (26.7, 57.5)
- moved NUMBERS 8.50 mm to (66.0, 57.5)
- moved IC1 8.50 mm to (66.0, 46.1)
- moved R1 8.50 mm to (44.5, 24.8)
- moved R10 8.50 mm to (23.4, 40.0)
- moved R11 8.50 mm to (15.2, 40.0)
- moved R12 8.50 mm to (7.11, 40.0)
- moved R13 8.50 mm to (45.7, 46.4)
- moved R14 8.50 mm to (38.1, 46.4)
- moved R15 8.50 mm to (30.0, 46.4)
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Connections:
- new net N$34: ESP-07/12.RESET, R20.1, RESET.1, RESET.2
- net +3V3: now also C5.+, R20.2
- net GND: now also C5.-, RESET.3, RESET.4
Routing:
- net GND: track 0.00 -> 266.1 mm
- net N$4: track 0.00 -> 104.1 mm
- net DIGIT_5: track 0.00 -> 101.0 mm
- net DIGIT_6: track 0.00 -> 92.6 mm
- net DIGIT_4: track 0.00 -> 89.6 mm
- net +3V3: track 0.00 -> 88.4 mm
- net DIGIT_1: track 0.00 -> 71.8 mm
- net DIGIT_2: track 0.00 -> 64.0 mm
- net DIGIT_3: track 0.00 -> 62.3 mm
- net +5V: track 0.00 -> 59.9 mm
- net N$34: track 0.00 -> 58.4 mm
- net NUM_B: track 0.00 -> 35.3 mm
- net +12V: track 0.00 -> 34.8 mm
- net NUM_A: track 0.00 -> 33.2 mm
- net NUM_C: track 0.00 -> 31.1 mm
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Other:
- board size 100 x 72 mm -> 100 x 63 mm
- board text added: "Tube+"
- board text removed: "Tube +"
