File: schematic/nixie board.sch (EAGLE design)
At the start: 56 parts, among them IC1 74141N, Q1 32,768kHz, Q2 16Mhz, T1 MPSA92, T10 MPSA92, T11 MPSA42, T12 MPSA92, T13 MPSA42, T14 MPSA92, T15 MPSA42, T16 MPSA42, T2 MPSA92, T3 MPSA42, T4 MPSA92, T5 MPSA42, T6 MPSA92, T7 MPSA42, T8 MPSA42, T9 MPSA92, U1 ATMEGA328P_PDIP

Commit message: Board Layout
Parts:
- removed BAT1: 3V, SparkFun-Electromechanical:BATTERY20PTH
- removed CHARACTERS: (no value), con-lstb:MA07-2
- removed ISP: (no value), con-lstb:MA03-2
- removed Q1: 32,768kHz, crystal:CRYSTALTC26V
- removed Q2: 16Mhz, crystal:CRYSTALHC49S
- removed R20, R21, R22: 470, resistor:R-EU_0204/7
- removed RN1, RN2: 33k, resistor-sil:E4R
- removed ROWS: (no value), con-lstb:MA05-2
- removed RTC: DS1307, ds1307_pcf8583:DS1307
- removed S1: Hour, switch-omron:10-XX
- removed S2: Minute, switch-omron:10-XX
- removed S3: Second, switch-omron:10-XX
- removed T13, T15, T16: MPSA42, transistor:MPSA42-NPN-TO92-EBC
- removed T14: MPSA92, transistor:MPSA92-PNP-TO92-EBC
- removed U1: ATMEGA328P_PDIP, SparkFun-DigitalIC:ATMEGA328P_PDIP
- added C3, C4: 1 µF, capacitor-wima:C5/4.5
- added DIGITS: (no value), con-lstb:MA03-2
- added ESP-07/12: ESP12, esp8266modules:ESP12
- added EXT1, EXT2: (no value), con-lsta:FE07-1
- added NUMBERS: (no value), con-lstb:MA05-2
- added PROG: (no value), switch-omron:10-XX
- added SR33: MCP1703-33, SteveMarple:MCP1702
- added SR50: MCP1703-50, SteveMarple:MCP1702
- C1, C2: value 22pf -> 1 µF; device SparkFun-Capacitors:CAPEZ -> capacitor-wima:C5/4.5
- R1, R2, R5: value 100k -> 33k; device resistor:R-EU_0207/2V -> resistor:R-EU_0204/7
- R11, R9: value 1k -> 470k
- R12, R7: value 100k -> 470k; device resistor:R-EU_0207/2V -> resistor:R-EU_0204/7
- R14, R16, R18: value 470k -> 100k; device resistor:R-EU_0204/7 -> resistor:R-EU_0207/2V
- R19: value 470k -> 10k; device resistor:R-EU_0204/7 -> resistor:R-EU_0207/2V
- R3, R6: value 470k -> 33k
- R4: value 1k -> 33k
- SERIAL: device con-lstb:MA04-1 -> con-lstb:MA05-1
- T1, T2, T4, T6: value MPSA92 -> MPSA42; device transistor:MPSA92-PNP-TO92-EBC -> transistor:MPSA42-NPN-TO92-EBC
- T11, T7, T8: value MPSA42 -> MPSA92; device transistor:MPSA42-NPN-TO92-EBC -> transistor:MPSA92-PNP-TO92-EBC
Connections:
- removed net N$34: CHARACTERS.1, IC1A.0
- removed net N$35: CHARACTERS.3, IC1A.8
- removed net N$36: CHARACTERS.5, IC1A.6
- removed net N$37: CHARACTERS.7, IC1A.4
- removed net N$38: CHARACTERS.9, IC1A.2
- removed net N$39: CHARACTERS.2, IC1A.9
- removed net N$40: CHARACTERS.4, IC1A.7
- removed net N$41: CHARACTERS.6, IC1A.5
- removed net N$42: CHARACTERS.8, IC1A.3
- removed net N$43: CHARACTERS.10, IC1A.1
- removed net N$44: C1.2, Q2.2, U1.PB6(XTAL1/TOSC1)
- removed net N$45: ISP.3, U1.PB5(SCK)
- removed net N$46: ISP.1, U1.PB4(MISO)
- removed net N$47: ISP.4, U1.PB3(MOSI/OC2)
- removed net N$48: R9.2, RTC.SDA, U1.PC4(ADC4/SDA)
- removed net N$49: R11.2, RTC.SCL, U1.PC5(ADC5/SCL)
- removed net N$50: Q1.2, RTC.X2
- removed net N$51: Q1.1, RTC.X1
- removed net N$52: C2.2, Q2.1, U1.PB7(XTAL2/TOSC2)
- removed net N$53: RN2D.1, U1.PD5(T1)
- removed net N$54: IC1A.C, U1.PC3(ADC3)
- removed net N$55: IC1A.D, U1.PD3(INT1)
- removed net N$56: IC1A.A, U1.PD4(XCK/T0)
- removed net N$57: IC1A.B, U1.PD2(INT0)
- removed net N$58: RN2C.1, U1.PD6(AIN0)
- removed net N$59: RN2B.1, U1.PD7(AIN1)
- removed net N$60: RN2A.1, U1.PB0(ICP)
- removed net N$61: RN1A.1, U1.PB1(OC1A)
- removed net N$62: RN1B.1, U1.PB2(SS/OC1B)
- removed net N$63: RN1C.1, U1.PC1(ADC1)
- removed net N$64: RN1D.1, U1.PC2(ADC2)
- removed net N$65: R22.2, R4.1, U1.PC0(ADC0)
- removed net N$66: BAT1.+, RTC.VBAT
- removed net N$67: SERIAL.2, U1.PD0(RXD)
- removed net N$68: SERIAL.1, U1.PD1(TXD)
- removed net N$72: ROWS.7, T9.C
- removed net RESET: ISP.5, U1.PC6(/RESET)
- removed net VCC: ISP.2, POWER.3, R11.1, R4.2, R9.1, RTC.VCC, SERIAL.3, U1.AREF, U1.AVCC, U1.VCC
- new net +12V: C1.1, C3.1, POWER.3, SR33.VIN, SR50.VIN
- new net +3V3: C4.1, ESP-07/12.CH_PD, ESP-07/12.VCC, EXT1.2, SERIAL.1, SR33.VOUT
- new net +5V: C2.1, EXT1.1, IC1P.VCC, SR50.VOUT
- new net DIGIT_1: ESP-07/12.RX, EXT2.1, R1.2, SERIAL.3
- new net DIGIT_2: ESP-07/12.GPIO4, EXT2.2, R2.2
- new net DIGIT_3: ESP-07/12.GPIO5, EXT2.3, R3.2
- new net DIGIT_4: ESP-07/12.GPIO0, EXT2.4, PROG.S, PROG.S1, R4.2
- new net DIGIT_5: ESP-07/12.GPIO2, EXT2.5, R5.2
- new net DIGIT_6: ESP-07/12.GPIO15, EXT2.6, R19.1, R6.2
- new net N$33: IC1A.9, NUMBERS.10
- new net NUM_A: ESP-07/12.GPIO13, EXT1.4, IC1A.A
- new net NUM_B: ESP-07/12.GPIO12, EXT1.5, IC1A.B
- new net NUM_C: ESP-07/12.GPIO14, EXT1.6, IC1A.C
- new net NUM_D: ESP-07/12.GPIO16, EXT1.7, IC1A.D
- net GND: now also C1.2, C2.2, C3.2, C4.2, ESP-07/12.GND, EXT1.3, IC1P.GND, PROG.P, PROG.P1, R19.2, SERIAL.5, SR33.GND, SR50.GND, T1.E, T2.E, T4.E, T6.E; no longer BAT1.-, C1.1, C2.1, CHARACTERS.13, CHARACTERS.14, ISP.6, RTC.GND, S1.P, S2.P, S3.P, SERIAL.4, T11.E, T13.E, T15.E, T16.E, T7.E, T8.E, U1.GND@1, U1.GND@2
- net N$1: now also ESP-07/12.TX, SERIAL.2; no longer RN1A.2, T3.B
- net N$10: now also IC1A.3, NUMBERS.4; no longer ROWS.8, T1.C
- net N$11: now also IC1A.5, NUMBERS.6; no longer R14.1, T11.C
- net N$12: now also R10.1, T4.C; no longer R8.1, T7.C
- net N$13: now also R10.2, R16.1, T10.B; no longer R5.1, R8.2, T4.B
- net N$14: now also IC1A.2, NUMBERS.3; no longer R12.1, R14.2, T9.B
- net N$15: now also DIGITS.6, T12.C; no longer ROWS.6, T2.C
- net N$16: now also R7.1, T1.C; no longer R16.1, T13.C
- net N$17: now also R8.1, T2.C; no longer R10.1, T8.C
- net N$18: now also R14.1, R8.2, T8.B; no longer R10.2, R7.1, T6.B
- net N$19: now also R7.2, T7.B; no longer R16.2, T10.B
- net N$2: now also IC1A.0, NUMBERS.1; no longer R3.1, T3.C
- net N$20: now also DIGITS.4, T10.C; no longer ROWS.4, T4.C
- net N$21: now also DIGITS.2, T8.C; no longer ROWS.2, T6.C
- net N$22: now also R9.1, T3.C; no longer R18.1, T15.C
- net N$23: now also R9.2, T9.B; no longer R18.2, T12.B
- net N$24: now also IC1A.4, NUMBERS.5; no longer R20.1, S1.S1
- net N$25: now also R11.1, T5.C; no longer R19.1, T16.C
- net N$26: now also R11.2, T11.B; no longer R19.2, T14.B
- net N$27: now also IC1A.6, NUMBERS.7; no longer R20.2, R21.1, S2.S1
- net N$28: now also IC1A.8, NUMBERS.9; no longer R21.2, R22.1, S3.S1
- net N$29: now also IC1A.7, NUMBERS.8; no longer RN2A.2, T11.B
- net N$3: now also IC1A.1, NUMBERS.2; no longer R1.1, R3.2, T1.B
- net N$30: now also R1.1, T1.B; no longer RN2B.2, T13.B
- net N$31: now also R3.1, T3.B; no longer RN2C.2, T15.B
- net N$32: now also R5.1, T5.B; no longer RN2D.2, T16.B
- net N$4: now also R14.2, R16.2, R18.2, T11.E, T7.E, T8.E; no longer R1.2, R12.2, R2.2, R5.2, R7.2, T1.E, T14.E, T2.E, T4.E, T6.E
- net N$5: now also R6.1, T6.B; no longer RN1B.2, T5.B
- net N$6: now also R4.1, T4.B; no longer RN1C.2, T7.B
- net N$69: now also DIGITS.5, T11.C; no longer ROWS.1, T14.C
- net N$7: now also R12.1, T6.C; no longer R6.1, T5.C
- net N$70: now also DIGITS.3, T9.C; no longer ROWS.3, T12.C
- net N$71: now also DIGITS.1, T7.C; no longer ROWS.5, T10.C
- net N$8: now also R12.2, R18.1, T12.B; no longer R2.1, R6.2, T2.B
- net N$9: now also R2.1, T2.B; no longer RN1D.2, T8.B
Other:
- note added: "Nixie Board"
- note added: "by Torsten Amshove"
- note added: "https://github.com/Torsten-/Arduino_NixieClock"
- note added: "v1.0"
- moved on the sheet: C1, C2, IC1, POWER, R1, R10, R11, R12, R13, R14, R15, R16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

Commit message: added reset and elko
Parts:
- added C5: 100 µF, rcl:CPOL-EUE2.5-6
- added R20: 10k, resistor:R-EU_0204/7
- added RESET: (no value), switch-omron:10-XX
- R19: device resistor:R-EU_0207/2V -> resistor:R-EU_0204/7
- SR33: value MCP1703-33 -> MCP1702-33
- SR50: value MCP1703-50 -> MCP1702-50
Connections:
- new net N$34: ESP-07/12.RESET, R20.1, RESET.S, RESET.S1
- net +3V3: now also C5.+, R20.2
- net GND: now also C5.-, RESET.P, RESET.P1
Other:
- moved on the sheet: ESP-07/12, EXT1, IC1, NUMBERS, SERIAL
